File: cm5/AlasIO/CM5IO.kicad_pcb (KiCad board)
At the start: 4 copper layers, 133.4 x 90 mm, 78 parts, among them J1 67910-5700, J14 JST_SHBM04B-SRSS-TB, J2 B2B-XH-A_LF__SN_, J4 0786463001, J5 USB_2_Vertical, J6 Conn_02x03_Counter_Clockwise, Q4 DTC143Z, U1 CAT24C128, U2 TLV320ADC6120IRTER, U5 74LVC1G07SE-7, U6 AP22653W6, U8 AP3441SHE-7B

Commit message: Way too much has changed...
Parts:
- added 48099-4000 : 480994000, KiCad:480994000, F.Cu at (222.2, 81.7)
- added J7: Conn_01x04, Connector_PinHeader_1.00mm:PinHeader_1x04_P1.00mm_Vertical, F.Cu at (203.0, 89.2)
- J5: value USB_2_Vertical -> USB3_A; footprint Connector_USB:C393950 -> Connector_USB:C168717
- moved C8 9.94 mm to (180.1, 138.7)
- moved C7 9.94 mm to (180.1, 141.1)
- moved J5 9.53 mm to (171.4, 151.7)
- moved J14 3.41 mm to (202.7, 80.5)
- moved Q4 2.33 mm to (204.5, 139.1)
- moved J1 1.71 mm to (222.2, 132.1)
- moved H6 0.51 mm to (234.8, 73.2)
Connections:
- J5 pad 2: /CM5_HighSpeed/USB3-0-D_N -> /CM5_HighSpeed/USB3-1-D_P
- J5 pad 3: /CM5_HighSpeed/USB3-0-D_P -> /CM5_HighSpeed/USB3-1-D_N
- J5 pad 5: /CM5_HighSpeed/VBUS -> /CM5_HighSpeed/USB3-1-RX_N
- J5 pad 6: /CM5_HighSpeed/USB3-1-D_N -> /CM5_HighSpeed/USB3-1-RX_P
- J5 pad 7: /CM5_HighSpeed/USB3-1-D_P -> GND
- J5 pad 8: GND -> /CM5_HighSpeed/USB3-1-TX_N
Routing:
- net /CM5_HighSpeed/USB3-1-D_P: track 72.5 -> 0.00 mm
- net /CM5_HighSpeed/USB3-1-D_N: track 70.5 -> 0.00 mm
- net /CM5_HighSpeed/USB3-0-D_N: track 55.3 -> 103.8 mm
- net /CM5_HighSpeed/USB3-0-D_P: track 55.0 -> 102.5 mm
- net /CM5_HighSpeed/VBUS: track 51.8 -> 22.2 mm, vias 1 -> 0
- net /CM5_GPIO ( Ethernet, GPIO, SDCARD)/PWM: track 32.7 -> 28.3 mm
- net /CM5_GPIO ( Ethernet, GPIO, SDCARD)/TACHO: track 43.7 -> 39.9 mm
- net /+5v: track 171.3 -> 168.0 mm, vias 3 -> 2
- net /CM5_HighSpeed/USB2_N: track 95.2 -> 97.3 mm
- net /PCIe-M2/W_DISABLE: track 33.0 -> 34.9 mm
- net /CM5_GPIO ( Ethernet, GPIO, SDCARD)/GPIO19: track 142.9 -> 144.9 mm
- added copper zone on B.Cu, net GND
- removed copper zone on B.Cu, net /CM5_HighSpeed/VBUS
Other:
- board size 133.4 x 90 mm -> 133.4 x 90.8 mm
