File: cm5/CM5IO_jake_v1/CM5IO-backups/CM5IO-2025-04-26_125745/CM5_HighSpeed.kicad_sch (KiCad schematic)
At the start: 9 parts, among them J5 USB3_A, J7 Conn_01x04, U6 AP22653W6

Commit message: Way too much has changed...
Parts:
- removed J5: USB3_A, Connector_USB:C168717, symbol Connector:USB3_A
- removed J7: Conn_01x04, Connector_PinHeader_1.00mm:PinHeader_1x04_P1.00mm_Vertical, symbol Connector_Generic:Conn_01x04
- added J12: USB3_A, CM5IO:MTCONN_UBAF30-D2011, symbol CM5IO:USB3_A
Connections:
- net GND: now also J12.10 (SHIELD), J12.A4 (GND), J12.A7 (DRAIN), J12.B4 (GND), J12.B7 (DRAIN)
- net USB3-0-D_N: now also J12.A2 (D-)
- net USB3-0-D_P: now also J12.A3 (D+)
- net USB3-0-RX_N: now also J12.A6 (SSRX+)
- net USB3-0-RX_P: now also J12.A5 (SSRX-)
- net USB3-0-TX_N: now also J12.A9 (SSTX+)
- net USB3-0-TX_P: now also J12.A8 (SSTX-)
- net USB3-1-D_N: now also J12.B2 (D-)
- net USB3-1-D_P: now also J12.B3 (D+)
- net USB3-1-RX_N: now also J12.B6 (SSRX+)
- net USB3-1-RX_P: now also J12.B5 (SSRX-)
- net USB3-1-TX_N: now also J12.B9 (SSTX+)
- net USB3-1-TX_P: now also J12.B8 (SSTX-)
- net VBUS: now also J12.A1 (VBUS), J12.B1 (VBUS)
Other:
- note added: "Stacked USB connectors"
- note added: "USB 3 Pairs P/N swapped to help routing"
