File: cm5/CM5IO_jake_v1/CM5IO-backups/CM5IO-2025-04-26_125745/PCIe-M2.kicad_sch (KiCad schematic)
At the start: 44 parts, among them J1 67910-5700, J4 0786463001, M1 M.2 Screw, M2 M.2 Solder Nut, M3 M.2 Solder Nut, M4 M.2 Solder Nut, M5 M.2 Solder Nut, Q4 DTC143Z, U1 CAT24C128, U8 AP3441SHE-7B

Commit message: Way too much has changed...
Parts:
- removed MolexClip1: ~, KiCad:480994000, symbol Interface:C492353
Connections:
- net USB_DN renamed USB_DM
Changed lines of the file:
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@@
 	(wire
 		(pts
-			(xy 177.8 41.91) (xy 176.53 41.91)
+			(xy 241.3 118.11) (xy 241.3 161.29)
 		)
 		(stroke
@@
 	(wire
 		(pts
-			(xy 241.3 118.11) (xy 241.3 161.29)
+			(xy 236.22 41.91) (xy 227.33 41.91)
 		)
 		(stroke
@@
 	(wire
 		(pts
-			(xy 236.22 41.91) (xy 227.33 41.91)
+			(xy 205.74 44.45) (xy 212.09 44.45)
 		)
 		(stroke
@@
 	(wire
 		(pts
-			(xy 176.53 41.91) (xy 176.53 44.45)
-		)
-		(stroke
-			(width 0)
-			(type default)
-		)
-	)
-	(wire
-		(pts
 			(xy 226.06 99.06) (xy 234.95 99.06)
 		)
@@
 	(wire
 		(pts
-			(xy 176.53 44.45) (xy 212.09 44.45)
-		)
-		(stroke
-			(width 0)
-			(type default)
-		)
-	)
-	(wire
-		(pts
 			(xy 207.01 87.63) (xy 212.09 87.63)
 		)
@@
 	(wire
 		(pts
-			(xy 176.53 46.99) (xy 176.53 49.53)
+			(xy 135.89 137.16) (xy 142.24 137.16)
 		)
 		(stroke
@@
 	(wire
 		(pts
-			(xy 135.89 137.16) (xy 142.24 137.16)
+			(xy 182.88 142.24) (xy 182.88 153.67)
 		)
 		(stroke
@@
 	(wire
 		(pts
-			(xy 182.88 142.24) (xy 182.88 153.67)
+			(xy 38.1 149.86) (xy 33.02 149.86)
 		)
 		(stroke
@@
 	(wire
 		(pts
-			(xy 38.1 149.86) (xy 33.02 149.86)
+			(xy 31.75 137.16) (xy 38.1 137.16)
 		)
 		(stroke
@@
 	(wire
 		(pts
-			(xy 31.75 137.16) (xy 38.1 137.16)
+			(xy 205.74 46.99) (xy 212.09 46.99)
 		)
 		(stroke
@@
 	(wire
 		(pts
-			(xy 176.53 46.99) (xy 212.09 46.99)
-		)
-		(stroke
-			(width 0)
-			(type default)
-		)
-	)
-	(wire
-		(pts
 			(xy 193.04 120.65) (xy 193.04 125.73)
 		)
@@
 		)
 	)
+	(label "USB_DP"
+		(at 205.74 44.45 180)
+		(effects
+			(font
+				(size 1.27 1.27)
+			)
+			(justify right bottom)
+		)
+	)
 	(label "UART_TX"
 		(at 231.14 74.93 0)
@@
 		)
 	)
+	(label "USB_DM"
+		(at 205.74 46.99 180)
+		(effects
+			(font
+				(size 1.27 1.27)
+			)
+			(justify right bottom)
+		)
+	)
 	(label "M2_3v3"
 		(at 276.86 46.99 0)
@@
 		)
 	)
-	(hierarchical_label "USB_DN"
-		(shape input)
-		(at 176.53 49.53 0)
-		(effects
-			(font
-				(size 1.27 1.27)
-			)
-			(justify left)
-		)
-	)
 	(hierarchical_label "EECLK"
 		(shape input)
@@
 		)
 	)
-	(hierarchical_label "USB_DP"
-		(shape input)
-		(at 177.8 41.91 0)
-		(effects
-			(font
-				(size 1.27 1.27)
-			)
-			(justify left)
-		)
-	)
 	(hierarchical_label "USER_BUTTON"
 		(shape output)
@@
 					(unit 1)
 				)
-			)
-		)
-	)
-	(symbol
-		(lib_id "Interface:C492353")
-		(at 181.61 20.32 0)
-		(unit 1)
-		(exclude_from_sim no)
-		(in_bom yes)
-		(on_board yes)
-		(dnp no)
-		(property "Reference" "MolexClip1"
-			(at 181.61 20.32 0)
-			(effects
-				(font
-					(size 1.27 1.27)
-				)
-			)
-		)
-		(property "Value" "~"
-			(at 182.245 16.51 0)
-			(effects
-				(font
-					(size 1.27 1.27)
-				)
-			)
-		)
-		(property "Footprint" "KiCad:480994000"
-			(at 181.61 20.32 0)
-			(effects
-				(font
-					(size 1.27 1.27)
-				)
-				(hide yes)
-			)
-		)
-		(property "Datasheet" ""
-			(at 181.61 20.32 0)
-			(effects
-				(font
-					(size 1.27 1.27)
-				)
-				(hide yes)
-			)
-		)
-		(property "Description" ""
-			(at 181.61 20.32 0)
-			(effects
-				(font
-					(size 1.27 1.27)
-				)
-				(hide yes)
-			)
-		)
-		(instances
-			(project ""
-				(path "/e63e39d7-6ac0-4ffd-8aa3-1841a4541b55/00000000-0000-0000-0000-00005ed4bb5b"
-					(reference "MolexClip1")
-					(unit 1)
-				)
