File: cm5/AlasIO/CM5IO-backups/CM5IO-2025-04-26_212721/CM5IO.kicad_pcb (KiCad board)
At the start: 4 copper layers, 133.4 x 90.8 mm, 80 parts, among them J1 67910-5700, J14 JST_SHBM04B-SRSS-TB, J2 B2B-XH-A_LF__SN_, J4 0786463001, J5 USB3_A, J6 Conn_02x03_Counter_Clockwise, J7 Conn_01x04, Q4 DTC143Z, U1 CAT24C128, U2 TLV320ADC6120IRTER, U5 74LVC1G07SE-7, U6 AP22653W6, U8 AP3441SHE-7B

Commit message: things are still not connected
Parts:
- removed J7: Conn_01x04, Connector_PinHeader_2.54mm:PinHeader_1x04_P2.54mm_Vertical
- J5: value USB3_A -> USB_2_Vertical; footprint Connector_USB:C168717 -> Connector_USB:C393950
- moved C8 9.94 mm to (170.1, 139.5)
- moved C7 9.94 mm to (170.2, 141.9)
- moved J5 9.53 mm to (165.0, 144.7), turned to 0 degrees
Connections:
- J5 pad 2: /CM5_HighSpeed/USB3-1-D_P -> /CM5_HighSpeed/USB3-0-D_N
- J5 pad 3: /CM5_HighSpeed/USB3-1-D_N -> /CM5_HighSpeed/USB3-0-D_P
- J5 pad 5: /CM5_HighSpeed/USB3-1-RX_N -> /CM5_HighSpeed/VBUS
- J5 pad 6: /CM5_HighSpeed/USB3-1-RX_P -> /CM5_HighSpeed/USB3-1-D_N
- J5 pad 7: GND -> /CM5_HighSpeed/USB3-1-D_P
- J5 pad 8: /CM5_HighSpeed/USB3-1-TX_N -> GND
Routing:
- net /+5v: track 98.2 -> 168.8 mm, vias 2 -> 3
- net /CM5_HighSpeed/USB3-1-TX_P: track 67.5 -> 0.00 mm
- net /CM5_HighSpeed/USB3-1-TX_N: track 66.3 -> 0.00 mm
- net /CM5_HighSpeed/USB3-1-RX_P: track 62.6 -> 0.00 mm
- net /CM5_HighSpeed/USB3-1-RX_N: track 62.4 -> 0.00 mm
- net /CM5_HighSpeed/VBUS: track 97.1 -> 51.8 mm
- net /CM5_HighSpeed/USB2_P: track 75.7 -> 116.6 mm
- net /CM5_HighSpeed/USB2_N: track 74.6 -> 95.2 mm
- net /CM5_HighSpeed/USB3-1-D_N: track 62.7 -> 70.5 mm
- net /CM5_HighSpeed/USB3-1-D_P: track 65.5 -> 72.5 mm
- net /CM5_HighSpeed/USB3-0-D_P: track 48.9 -> 55.0 mm
- net /CM5_HighSpeed/USB3-0-D_N: track 50.9 -> 55.3 mm
- net /CM5_GPIO ( Ethernet, GPIO, SDCARD)/GPIO15: track 52.8 -> 53.8 mm
- added copper zone on B.Cu, net /CM5_HighSpeed/VBUS
