File: cm5/CM5IO.kicad_sch (KiCad schematic)
At the start: 11 parts, among them J2 B2B-XH-A_LF__SN_

Commit message: Hopefully these are the corrected parts, need to cross-reference the BOM to what was ordered
Other:
- company: E-SMART SOLUTIONS -> Ridgeline Radio
- title: Compute Module 5 IO -> Alas Compute Module 5 IO
Changed lines of the file:
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@@
 	(paper "A4")
 	(title_block
-		(title "Compute Module 5 IO")
+		(title "Alas Compute Module 5 IO")
 		(rev "1")
-		(company "E-SMART SOLUTIONS")
-		(comment 1 "Mostafa Bkair")
+		(company "Ridgeline Radio")
+		(comment 1 "Jake Wood")
 	)
 	(text "Connectors\n-------\nEthernet\nSDCARD\n40way RPI\nJumpers\nFan\nBattery"

Commit message: Uh in this version, I have made the 5v trace fatter
Other:
- sheet CM5_GPIO ( Ethernet, GPIO, SDCARD) ports: added none; removed USER_LED
Changed lines of the file:
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@@
-	(wire
-		(pts
-			(xy 186.69 72.39) (xy 214.63 72.39)
-		)
-		(stroke
-			(width 0)
-			(type default)
-		)
-	)
 	(wire
 		(pts
@@
 	(wire
 		(pts
-			(xy 146.05 172.72) (xy 146.05 157.48)
-		)
-		(stroke
-			(width 0)
-			(type default)
-		)
-	)
-	(wire
-		(pts
 			(xy 134.62 96.52) (xy 134.62 111.76)
 		)
@@
 	(wire
 		(pts
-			(xy 208.28 83.82) (xy 208.28 172.72)
-		)
-		(stroke
-			(width 0)
-			(type default)
-		)
-	)
-	(wire
-		(pts
-			(xy 208.28 172.72) (xy 146.05 172.72)
-		)
-		(stroke
-			(width 0)
-			(type default)
-		)
-	)
-	(wire
-		(pts
 			(xy 204.47 48.26) (xy 214.63 48.26)
 		)
@@
 	(wire
 		(pts
-			(xy 204.47 81.28) (xy 204.47 163.83)
-		)
-		(stroke
-			(width 0)
-			(type default)
-		)
-	)
-	(wire
-		(pts
 			(xy 149.86 170.18) (xy 241.3 170.18)
 		)
@@
 	(wire
 		(pts
-			(xy 214.63 81.28) (xy 204.47 81.28)
-		)
-		(stroke
-			(width 0)
-			(type default)
-		)
-	)
-	(wire
-		(pts
 			(xy 162.56 96.52) (xy 162.56 111.76)
 		)
@@
 	(wire
 		(pts
-			(xy 214.63 83.82) (xy 208.28 83.82)
-		)
-		(stroke
-			(width 0)
-			(type default)
-		)
-	)
-	(wire
-		(pts
 			(xy 232.41 86.36) (xy 232.41 168.91)
 		)
@@
 	(wire
 		(pts
-			(xy 168.91 163.83) (xy 204.47 163.83)
-		)
-		(stroke
-			(width 0)
-			(type default)
-		)
-	)
-	(wire
-		(pts
 			(xy 186.69 125.73) (xy 195.58 125.73)
-		)
-		(stroke
-			(width 0)
-			(type default)
-		)
-	)
-	(wire
-		(pts
-			(xy 168.91 163.83) (xy 168.91 157.48)
 		)
 		(stroke
@@
 			)
 		)
-		(pin "USER_LED" input
-			(at 168.91 157.48 270)
-			(effects
-				(font
-					(size 1.27 1.27)
-				)
-				(justify left)
-			)
-		)
 		(pin "UART_TX" input
 			(at 165.1 157.48 270)
@@
 		)
 		(pin "PCIE_PWR_EN" input
-			(at 214.63 72.39 180)
+			(at 214.63 62.23 180)
 			(effects
 				(font
@@
 		)
 		(pin "EECLK" input
-			(at 214.63 83.82 180)
+			(at 214.63 68.58 180)
 			(effects
 				(font
@@
 		)
 		(pin "USER_LED" input
-			(at 214.63 81.28 180)
-			(effects
-				(font
+			(at 214.63 66.04 180)
+			(effects
+				(font
