File: cm5/CM5IO-backups/CM5IO-2025-05-01_222343/CM5IO.kicad_sch (KiCad schematic)
At the start: 11 parts, among them J2 B2B-XH-A_LF__SN_

Commit message: Delete some unnecessary components and fix up some of the trace thicknesses
Other:
- sheet CM5_GPIO ( Ethernet, GPIO, SDCARD) ports: added USER_LED; removed none
Changed lines of the file:
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@@
+	(wire
+		(pts
+			(xy 186.69 72.39) (xy 214.63 72.39)
+		)
+		(stroke
+			(width 0)
+			(type default)
+		)
+	)
 	(wire
 		(pts
@@
 	(wire
 		(pts
-			(xy 186.69 72.39) (xy 200.66 72.39)
+			(xy 146.05 172.72) (xy 146.05 157.48)
 		)
 		(stroke
@@
 	(wire
 		(pts
+			(xy 208.28 83.82) (xy 208.28 172.72)
+		)
+		(stroke
+			(width 0)
+			(type default)
+		)
+	)
+	(wire
+		(pts
+			(xy 208.28 172.72) (xy 146.05 172.72)
+		)
+		(stroke
+			(width 0)
+			(type default)
+		)
+	)
+	(wire
+		(pts
 			(xy 204.47 48.26) (xy 214.63 48.26)
 		)
@@
 	(wire
 		(pts
-			(xy 200.66 62.23) (xy 214.63 62.23)
-		)
-		(stroke
-			(width 0)
-			(type default)
-		)
-	)
-	(wire
-		(pts
 			(xy 92.71 101.6) (xy 104.14 101.6)
 		)
@@
 	(wire
 		(pts
+			(xy 204.47 81.28) (xy 204.47 163.83)
+		)
+		(stroke
+			(width 0)
+			(type default)
+		)
+	)
+	(wire
+		(pts
 			(xy 149.86 170.18) (xy 241.3 170.18)
 		)
@@
 	(wire
 		(pts
+			(xy 214.63 81.28) (xy 204.47 81.28)
+		)
+		(stroke
+			(width 0)
+			(type default)
+		)
+	)
+	(wire
+		(pts
 			(xy 162.56 96.52) (xy 162.56 111.76)
 		)
@@
 	(wire
 		(pts
-			(xy 200.66 72.39) (xy 200.66 62.23)
-		)
-		(stroke
-			(width 0)
-			(type default)
-		)
-	)
-	(wire
-		(pts
 			(xy 129.54 50.8) (xy 120.65 50.8)
 		)
@@
 	(wire
 		(pts
+			(xy 214.63 83.82) (xy 208.28 83.82)
+		)
+		(stroke
+			(width 0)
+			(type default)
+		)
+	)
+	(wire
+		(pts
 			(xy 232.41 86.36) (xy 232.41 168.91)
 		)
@@
 	(wire
 		(pts
+			(xy 168.91 163.83) (xy 204.47 163.83)
+		)
+		(stroke
+			(width 0)
+			(type default)
+		)
+	)
+	(wire
+		(pts
 			(xy 186.69 125.73) (xy 195.58 125.73)
+		)
+		(stroke
+			(width 0)
+			(type default)
+		)
+	)
+	(wire
+		(pts
+			(xy 168.91 163.83) (xy 168.91 157.48)
 		)
 		(stroke
@@
 			)
 		)
+		(pin "USER_LED" input
+			(at 168.91 157.48 270)
+			(effects
+				(font
+					(size 1.27 1.27)
+				)
+				(justify left)
+			)
+		)
 		(pin "UART_TX" input
 			(at 165.1 157.48 270)
@@
 		)
 		(pin "PCIE_PWR_EN" input
-			(at 214.63 62.23 180)
+			(at 214.63 72.39 180)
 			(effects
 				(font
@@
 		)
 		(pin "EECLK" input
-			(at 214.63 68.58 180)
+			(at 214.63 83.82 180)
 			(effects
 				(font
@@
 		)
 		(pin "USER_LED" input
-			(at 214.63 66.04 180)
-			(effects
-				(font
+			(at 214.63 81.28 180)
+			(effects
+				(font
